File: GP2040-RE/GP2040-RE.kicad_sch (KiCad schematic)
At the start: 41 parts, among them J1 I2C Slave, J2 DEBUG, J3 USB Programming, J4 Console, J5 ManualConsoleSelection, J6 I2C Passthrough, J7 Micro_SD_Card, SW1 BOOTSEL, SW2 RESET, U1 W25Q16JV, U2 RP2040, U3 RT6154AGQW

Commit message: Much happier now
Parts:
- removed J5: ManualConsoleSelection, Connector_PinHeader_2.54mm:PinHeader_2x04_P2.54mm_Vertical, symbol Connector_Generic:Conn_02x04_Odd_Even
- added J5: RJ-45, RJ-45:CONN8_2-908LF_AMP, symbol RJ-45:54602-908LF
- added J8: Conn_01x10, Connector_PinHeader_2.54mm:PinHeader_1x10_P2.54mm_Vertical, symbol Connector_Generic:Conn_01x10
- J1, J6: footprint Connector_JST:JST_PH_S4B-PH-K_1x04_P2.00mm_Horizontal -> JST-SH:JST_SH_SM04B-SRSS-TB_1x04-1MP_P1.00mm_Horizontal; symbol Connector:Conn_01x04_Pin -> JST-SH:SM04B-SRSS-TB
- J2: footprint Connector_PinHeader_2.54mm:PinHeader_1x03_P2.54mm_Vertical -> JST-SH:JST_SH_SM03B-SRSS-TB_1x03-1MP_P1.00mm_Horizontal
- J7: footprint Connector_Card:microSD_HC_Molex_47219-2001 -> microSD:MEM2061-01-188-00-A_GCT; symbol Connector:Micro_SD_Card_Det1 -> microSD:MEM2061-01-188-00-A
- S1: renamed from SW1; footprint Button_Switch_SMD:SW_SPST_B3S-1000 -> EVP_BB2A9B000:SW_EVP-BB2A9B000; symbol Switch:SW_Push -> EVP-BB2A9B000:EVP-BB2A9B000; ARROW_ELECTRONICS-PURCHASE-URL (none) -> https://snapeda.com/shop?store=Arrow+Electronics&id=584571; DIGI-KEY_PART_NUMBER (none) -> P19888CT-ND; DIGIKEY-PURCHASE-URL (none) -> https://snapeda.com/shop?store=DigiKey&id=584571; MAXIMUM_PACKAGE_HEIGHT (none) -> 0.58mm; MF (none) -> Panasonic Electronic; MOUSER-PURCHASE-URL (none) -> https://snapeda.com/shop?store=Mouser&id=584571; MP (none) -> EVP-BB2A9B000; PACKAGE (none) -> None
- S2: renamed from SW2; footprint Button_Switch_SMD:SW_SPST_B3S-1000 -> EVP_BB2A9B000:SW_EVP-BB2A9B000; symbol Switch:SW_Push -> EVP-BB2A9B000:EVP-BB2A9B000; ARROW_ELECTRONICS-PURCHASE-URL (none) -> https://snapeda.com/shop?store=Arrow+Electronics&id=584571; DIGI-KEY_PART_NUMBER (none) -> P19888CT-ND; DIGIKEY-PURCHASE-URL (none) -> https://snapeda.com/shop?store=DigiKey&id=584571; MAXIMUM_PACKAGE_HEIGHT (none) -> 0.58mm; MF (none) -> Panasonic Electronic; MOUSER-PURCHASE-URL (none) -> https://snapeda.com/shop?store=Mouser&id=584571; MP (none) -> EVP-BB2A9B000; PACKAGE (none) -> None
- U1: footprint Package_SO:SOIC-8_5.23x5.23mm_P1.27mm -> W25Q16:USON-8_UX_2x3x0p6_WIN
Connections:
- net +3.3V: now also J7.P4 (VDD), J8.2 (Pin_2); no longer J7.4 (VDD)
- net BlueSolid: now also J5.4
- net BlueStripe: now also J5.5
- net BrownSolid: now also J5.8
- net BrownStripe: now also J5.7
- net CD_gpio: now also J7.10 (CARD_DETECT)
- net CLK_gpio: now also J7.P5 (CLK); no longer J7.5 (CLK)
- net CMD_gpio: now also J7.P3 (CMD); no longer J7.3 (CMD)
- net D0_gpio: now also J7.P7 (DAT0); no longer J7.7 (DAT0)
- net D1_gpio: now also J7.P8 (DAT1); no longer J7.8 (DAT1)
- net D2_gpio: now also J7.P1 (DAT2); no longer J7.1 (DAT2)
- net D3_gpio: now also J7.P2 (CD/DAT3); no longer J7.2 (DAT3/CD)
- net GND: now also J7.11 (GROUND), J7.12 (GROUND), J7.P6 (VSS), S1.A1, S1.A2, S2.A1, S2.A2, J5.1, J8.1 (Pin_1); no longer J7.10 (SHIELD), J7.6 (VSS), S1.1, S2.1
- net GreenSolid: now also J5.6
- net GreenStripe: now also J5.3
- net OrangeSolid: now also J5.2
- net RUN: now also S2.B1, S2.B2; no longer S2.2
- net at R1.1: now also S1.B1, S1.B2; no longer S1.2
- net SPI1_CSn: now reaches U2.16 (GPIO13)
- net OCS: now reaches U2.34 (GPIO22)
- net OCS: now also J8.4 (Pin_4)
- net RESET: now reaches U2.35 (GPIO23)
- net RESET: now also J8.5 (Pin_5)
- net Data_Command: now reaches U2.36 (GPIO24)
- net Data_Command: now also J8.6 (Pin_6)
- net SPI1_SCK: now reaches U2.38 (GPIO26_ADC0)
- net SPI1_SCK: now also J8.7 (Pin_7)
- net SPI1_TX_MOSI: now reaches U2.39 (GPIO27_ADC1)
- net SPI1_TX_MOSI: now also J8.8 (Pin_8)
- net SPI1_RX_MISO: now reaches U2.40 (GPIO28_ADC2)
- net SPI1_RX_MISO: now also J8.9 (Pin_9)
- net GC: no longer names the net of U2.14 (GPIO11)
- net N64: no longer names the net of U2.13 (GPIO10)
- net NES: no longer names the net of U2.11 (GPIO8)
- net SNES: no longer names the net of U2.12 (GPIO9)
- no-connect marks 14 -> 13
Other:
- moved on the sheet: J2, J3, J4, R1

Commit message: Now with blinky lights
Parts:
- added D3, D4: LED_Small, LED_SMD:LED_0201_0603Metric, symbol Device:LED_Small
- added Q1: SBC846BWT1G, SBC846BW:SOT-323-3_2P2X1P35_ONS, symbol SBC846BW:SBC846BWT1G
- added R10, R11, R12: 10k, Resistor_SMD:R_0201_0603Metric, symbol Device:R_Small
- added U4: TPS3702CX50DDCR, TPS3702CX50:DDC0006A_N, symbol TPS3702CX50:TPS3702CX50DDCR
Connections:
- net +3.3V: now also R10.1, R12.1, U4.5 (VDD); no longer J8.2 (Pin_2)
- net GND: now also D3.1 (K), D4.1 (K), U4.2 (GND), U4.4 (SET)
- net VBUS: now also Q1.3 (C)
- net InputVoltage: now reaches D1.1, D2.1, R9.2, U3.10 (VIN), U3.11 (VIN)
- net InputVoltage: now also U4.3 (SENSE)
- new net: D4.2 (A), R11.2
- new net: D3.2 (A), R12.2
- new net: J8.2 (Pin_2), Q1.2 (E)
- new net 5V_EN: Q1.1 (B), R10.2, R11.1, U4.1 (OUTA_N), U4.6 (OUTB_N)
Other:
- moved on the sheet: J8
