File: GP2040-RE/GP2040-RE.kicad_sch (KiCad schematic)
At the start: 49 parts, among them J1 I2C Slave, J2 DEBUG, J3 USB Programming, J4 Console, J5 RJ-45, J6 I2C Passthrough, J7 Micro_SD_Card, J8 Conn_01x10, Q1 SBC846BWT1G, U1 W25Q16JV, U2 RP2040, U3 RT6154AGQW, U4 TPS3702CX50DDCR

Commit message: rebuilding part libraries
Parts:
- added C?: 0.1uF, symbol Device:C_Small
- C?: renamed from C13; footprint Capacitor_SMD:C_0201_0603Metric -> Capacitor_SMD:C_0603_1608Metric
- C?: renamed from C10; footprint Capacitor_SMD:C_0201_0603Metric -> Capacitor_SMD:C_0603_1608Metric
- C?: renamed from C16; footprint Capacitor_SMD:C_0201_0603Metric -> Capacitor_SMD:C_0603_1608Metric
- C?: renamed from C14; footprint Capacitor_SMD:C_0201_0603Metric -> Capacitor_SMD:C_0603_1608Metric
- C?: renamed from C7; footprint Capacitor_SMD:C_0201_0603Metric -> Capacitor_SMD:C_0603_1608Metric
- C?: renamed from C6; footprint Capacitor_SMD:C_0201_0603Metric -> Capacitor_SMD:C_0603_1608Metric
- C?: renamed from C3; footprint Capacitor_SMD:C_0201_0603Metric -> Capacitor_SMD:C_0603_1608Metric
- C?: renamed from C12; footprint Capacitor_SMD:C_0201_0603Metric -> Capacitor_SMD:C_0603_1608Metric
- C?: renamed from C9; footprint Capacitor_SMD:C_0201_0603Metric -> Capacitor_SMD:C_0603_1608Metric
- C?: renamed from C15; footprint Capacitor_SMD:C_0201_0603Metric -> Capacitor_SMD:C_0603_1608Metric
- C?: renamed from C8; footprint Capacitor_SMD:C_0201_0603Metric -> Capacitor_SMD:C_0603_1608Metric
- C?: renamed from C2; footprint Capacitor_SMD:C_0201_0603Metric -> Capacitor_SMD:C_0603_1608Metric
- C?: renamed from C5; footprint Capacitor_SMD:C_0201_0603Metric -> Capacitor_SMD:C_0603_1608Metric
- C?: renamed from C1; footprint Capacitor_SMD:C_0201_0603Metric -> Capacitor_SMD:C_0603_1608Metric
- C?: renamed from C11; footprint Capacitor_SMD:C_0201_0603Metric -> Capacitor_SMD:C_0603_1608Metric
- C?: renamed from C4; footprint Capacitor_SMD:C_0201_0603Metric -> Capacitor_SMD:C_0603_1608Metric
- D?: renamed from D3; footprint LED_SMD:LED_0201_0603Metric -> LED_SMD:LED_0603_1608Metric
- D?: renamed from D4; footprint LED_SMD:LED_0201_0603Metric -> LED_SMD:LED_0603_1608Metric
- R?: renamed from R10; footprint Resistor_SMD:R_0201_0603Metric -> Resistor_SMD:R_0603_1608Metric
- R?: renamed from R5; footprint Resistor_SMD:R_0201_0603Metric -> Resistor_SMD:R_0603_1608Metric
- R?: renamed from R11; footprint Resistor_SMD:R_0201_0603Metric -> Resistor_SMD:R_0603_1608Metric
- R?: renamed from R2; footprint Resistor_SMD:R_0201_0603Metric -> Resistor_SMD:R_0603_1608Metric
- R?: renamed from R4; footprint Resistor_SMD:R_0201_0603Metric -> Resistor_SMD:R_0603_1608Metric
- R?: renamed from R8; footprint Resistor_SMD:R_0201_0603Metric -> Resistor_SMD:R_0603_1608Metric
- R?: renamed from R7; footprint Resistor_SMD:R_0201_0603Metric -> Resistor_SMD:R_0603_1608Metric
- R?: renamed from R1; footprint Resistor_SMD:R_0201_0603Metric -> Resistor_SMD:R_0603_1608Metric
- R?: renamed from R9; footprint Resistor_SMD:R_0201_0603Metric -> Resistor_SMD:R_0603_1608Metric
- R?: renamed from R12; footprint Resistor_SMD:R_0201_0603Metric -> Resistor_SMD:R_0603_1608Metric
- R?: renamed from R6; footprint Resistor_SMD:R_0201_0603Metric -> Resistor_SMD:R_0603_1608Metric
- R?: renamed from R3; footprint Resistor_SMD:R_0201_0603Metric -> Resistor_SMD:R_0603_1608Metric
- U?: renamed from U2; footprint Package_DFN_QFN:QFN-56-1EP_7x7mm_P0.4mm_EP3.2x3.2mm -> GP2040-RE:QFN56_7X7_RPI; symbol MCU_RaspberryPi:RP2040 -> GP2040-RE:RP2040; DigiKey Part Number (none) -> 2648-SC0914(13)CT-ND
- renumbered D1 to D?, D2 to D?, J3 to J?, J7 to J?, J4 to J?, J2 to J?, J1 to J?, J6 to J?, J5 to J?, J8 to J?, L1 to L?, Q1 to Q?, S1 to S?, S2 to S?, U1 to U?, U3 to U?, U4 to U?, XTAL1 to XTAL?
Connections:
- net +: no longer R?.2, U?.47 (USB_DP)
- net +1V1: no longer U?.23 (DVDD), U?.45 (VREG_VOUT), U?.50 (DVDD)
- net +3.3V: now also C?.1; no longer U?.1 (IOVDD), U?.10 (IOVDD), U?.22 (IOVDD), U?.33 (IOVDD), U?.42 (IOVDD), U?.43 (ADC_AVDD), U?.44 (VREG_IN), U?.48 (USB_VDD), U?.49 (IOVDD)
- net BlueSolid: no longer U?.6 (GPIO4)
- net BlueStripe: no longer U?.7 (GPIO5)
- net BrownStripe: no longer U?.9 (GPIO7)
- net CD_gpio: no longer U?.18 (GPIO15)
- net CLK_gpio: no longer U?.27 (GPIO16)
- net CMD_gpio: no longer U?.28 (GPIO17)
- net D+: now also R?.2; no longer R?.1
- net D-: now also R?.2; no longer R?.1
- net D0_gpio: no longer U?.29 (GPIO18)
- net D1_gpio: no longer U?.30 (GPIO19)
- net D2_gpio: no longer U?.31 (GPIO20)
- net D3_gpio: no longer U?.32 (GPIO21)
- net Data_Command: no longer U?.36 (GPIO24)
- net GND: now also C?.2; no longer U?.19 (TESTEN), U?.57 (GND)
- net GreenSolid: no longer U?.8 (GPIO6)
- net GreenStripe: no longer U?.5 (GPIO3)
- net OCS: no longer U?.34 (GPIO22)
- net OrangeSolid: no longer U?.4 (GPIO2)
- net QSPI_SCLK: no longer U?.52 (QSPI_SCLK)
- net QSPI_SD0: no longer U?.53 (QSPI_SD0)
- net QSPI_SD1: no longer U?.55 (QSPI_SD1)
- net QSPI_SD2: no longer U?.54 (QSPI_SD2)
- net QSPI_SD3: no longer U?.51 (QSPI_SD3)
- net QSPI_SS: no longer U?.56 (QSPI_SS)
- net RESET: no longer U?.35 (GPIO23)
- net RUN: no longer U?.26 (RUN)
- net SCL: no longer U?.3 (GPIO1)
- net SDA: no longer U?.2 (GPIO0)
- net SPI1_CSn: no longer U?.16 (GPIO13)
- net SPI1_RX_MISO: no longer U?.40 (GPIO28_ADC2)
- net SPI1_SCK: no longer U?.38 (GPIO26_ADC0)
- net SPI1_TX_MOSI: no longer U?.39 (GPIO27_ADC1)
- net SWCLK: no longer U?.24 (SWCLK)
- net SWDIO: no longer U?.25 (SWD)
- net XIN: no longer U?.20 (XIN)
- net -: no longer names the net of U?.46 (USB_DM)
- net -: now also R?.1; no longer R?.2
- new net: R?.1, U?.47 (USB_DP)
Other:
- note removed: "Ensure C3 is close to Pin 45 on the RP2040"
- note removed: "Ensure C7 is close to Pin 44 on the RP2040"
- moved on the sheet: C?, R?

Commit message: 4 Layer board
Parts:
- removed C?: 1uF, Capacitor_SMD:C_0603_1608Metric, symbol Device:C_Small
- removed J?: Console, Connector_PinHeader_2.54mm:PinHeader_1x08_P2.54mm_Vertical, symbol Connector:Conn_01x08_Pin
- added C13: 2.2u 6.3V X5R 20%, Capacitor_SMD:C_0603_1608Metric, symbol Device:C_Small
- added C18: 47u 6.3V X5R 20%, Capacitor_SMD:C_0603_1608Metric, symbol Device:C_Small
- added J5: Conn_01x03, Connector_PinHeader_2.54mm:PinHeader_1x03_P2.54mm_Vertical, symbol Connector_Generic:Conn_01x03
- added R11: VREF SHUNT 2%, GP2040-RE:DBZ3, symbol GP2040-RE:VREF
- C1: renamed from C?; value 2.2u 6.3v 20% -> 2.2u 6.3V X5R 20%; DigiKey Part Number (none) -> 587-MCASJ168SB5225MTNA01CT-ND
- C10, C11, C15, C2, C4, C5, C6, C7, C8, C9: renamed from C?; value 100n 6.3V 10% -> 100n 6.3V X5R 10%; DigiKey Part Number (none) -> 399-17575-1-ND
- C12: renamed from C?; value 100n 6.3V 10% -> 2.2u 6.3V X5R 20%; DigiKey Part Number (none) -> 587-MCASJ168SB5225MTNA01CT-ND
- C14: renamed from C?; value 1uF -> 2.2u 6.3V X5R 20%; DigiKey Part Number (none) -> 587-MCASJ168SB5225MTNA01CT-ND
- C16, C17: renamed from C?; value 47u 6.3V 20% -> 47u 6.3V X5R 20%; DigiKey Part Number (none) -> 1276-CL10A476MQ8QRNCCT-ND
- C3: renamed from C?; value 0.1uF -> 100n 6.3V X5R 10%; footprint (none) -> Capacitor_SMD:C_0603_1608Metric; DigiKey Part Number (none) -> 399-17575-1-ND
- D1, D2: renamed from D?; DigiKey Part Number (none) -> 3147-B1931NG--20D001114U1930CT-ND
- D3, D4: renamed from D?; value MBR120VLSFT1G -> 20V 1A; footprint MBR120V:SDO_SOD-123FL_ONS -> GP2040-RE:SDO_SOD-123FL_ONS; symbol MBR120V:MBR120VLSFT1G -> GP2040-RE:Schottky; DigiKey Part Number (none) -> MBR120VLSFT1GOSCT-ND
- J1: renamed from J?; value I2C Slave -> I2C Target; footprint JST-SH:JST_SH_SM04B-SRSS-TB_1x04-1MP_P1.00mm_Horizontal -> GP2040-RE:CONN_SM04B-SRSS-TB_JST; symbol JST-SH:SM04B-SRSS-TB -> GP2040-RE:qwiic; DigiKey Part Number (none) -> 455-SM04B-SRSS-TBCT-ND
- J2: renamed from J?; value I2C Passthrough -> I2C Controller; footprint JST-SH:JST_SH_SM04B-SRSS-TB_1x04-1MP_P1.00mm_Horizontal -> GP2040-RE:CONN_SM04B-SRSS-TB_JST; symbol JST-SH:SM04B-SRSS-TB -> GP2040-RE:qwiic; DigiKey Part Number (none) -> 455-SM04B-SRSS-TBCT-ND
- J3: renamed from J?; value DEBUG -> SM03B-SRSS-TB_LF__SN_; footprint JST-SH:JST_SH_SM03B-SRSS-TB_1x03-1MP_P1.00mm_Horizontal -> GP2040-RE:JST_SM03B-SRSS-TB_LF__SN_; symbol Connector:Conn_01x03_Pin -> GP2040-RE:SM03B-SRSS-TB_LF__SN_; DigiKey Part Number (none) -> 455-BM03B-SRSS-TBTCT-ND; MANUFACTURER (none) -> JST; MP (none) -> SM03B-SRSS-TB(LF)(SN); SnapEDA_Link (none) -> https://www.snapeda.com/parts/SM03B-SRSS-TB(LF)(SN)/JST+Sal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
- J4: renamed from J?; DigiKey Part Number (none) -> 2057-PH1-04-UA-ND
- J6: renamed from J?; value Micro_SD_Card -> microSD; footprint microSD:MEM2061-01-188-00-A_GCT -> GP2040-RE:MEM2061-01-188-00-A_GCT; symbol microSD:MEM2061-01-188-00-A -> GP2040-RE:microSD; DigiKey Part Number (none) -> 2073-MEM2061-01-188-00-ACT-ND
- J7: renamed from J?; footprint RJ-45:CONN8_2-908LF_AMP -> GP2040-RE:CONN8_2-908LF_AMP; symbol RJ-45:54602-908LF -> GP2040-RE:RJ-45; DigiKey Part Number (none) -> 2057-MTJ-889X1-ND
- J8: renamed from J?; DigiKey Part Number (none) -> SAM1112-10-ND
- L1: renamed from L?; value 1uH -> SRN2512-1R0M; footprint SRN2512:IND_SRN2512_BRN -> GP2040-RE:IND_SRN2512_BRN; symbol SRN2512:SRN2512-1R0M -> GP2040-RE:SRN2512-1R0M; DigiKey Part Number (none) -> SRN2512-1R0MCT-ND
- Q1: renamed from Q?; value SBC846BWT1G -> NPN 65V 0.1A; footprint SBC846BW:SOT-323-3_2P2X1P35_ONS -> GP2040-RE:SOT-323-3_2P2X1P35_ONS; symbol SBC846BW:SBC846BWT1G -> GP2040-RE:FET; DigiKey Part Number (none) -> SBC846BWT1GOSCT-ND
- R1: renamed from R?; DigiKey Part Number (none) -> P1.00KHCT-ND
- R10, R4, R5: renamed from R?; DigiKey Part Number (none) -> P10.0KHCT-ND
- R12, R13: renamed from R?; value 27 50mW 1% -> 27 50mW 1% M0603; DigiKey Part Number (none) -> P27.0HCT-ND
- R2, R3: renamed from R?; DigiKey Part Number (none) -> P4.70KHCT-ND
- R6, R7, R9: renamed from R?; DigiKey Part Number (none) -> P100KHCT-ND
- R8: renamed from R?; DigiKey Part Number (none) -> P560KHCT-ND
- S1: renamed from S?; value BOOTSEL -> Buttons; footprint EVP_BB2A9B000:SW_EVP-BB2A9B000 -> GP2040-RE:SW_EVP-BB2A9B000; symbol EVP-BB2A9B000:EVP-BB2A9B000 -> GP2040-RE:Buttons; DigiKey Part Number (none) -> P19888CT-ND
- S2: renamed from S?; value RESET -> Buttons; footprint EVP_BB2A9B000:SW_EVP-BB2A9B000 -> GP2040-RE:SW_EVP-BB2A9B000; symbol EVP-BB2A9B000:EVP-BB2A9B000 -> GP2040-RE:Buttons; DigiKey Part Number (none) -> P19888CT-ND
- U2: renamed from U?; value W25Q16JV -> 16M; footprint W25Q16:USON-8_UX_2x3x0p6_WIN -> GP2040-RE:USON-8_UX_2x3x0p6_WIN; symbol W25Q16JVUXIQ:W25Q16JV -> GP2040-RE:Flash Memory; DigiKey Part Number (none) -> 256-W25Q16JVUXIQTRCT-ND
- U4: renamed from U?; value RT6154AGQW -> Linear Regulator; footprint RT6154A:QFN_4AGQW_RIT -> GP2040-RE:QFN_4AGQW_RIT; symbol RT6154A:RT6154AGQW -> GP2040-RE:Linear Regulator; DigiKey Part Number (none) -> 1028-1338-1-ND
- U5: renamed from U?; footprint TPS3702CX50:DDC0006A_N -> GP2040-RE:DDC0006A_N; symbol TPS3702CX50:TPS3702CX50DDCR -> GP2040-RE:Voltage Supervisor; DigiKey Part Number (none) -> 296-TPS3702CX50DDCRCT-ND
- XTAL1: renamed from XTAL?; footprint SIT1602:SON4_SIT1602-3_SIT -> GP2040-RE:SON4_SIT1602-3_SIT; symbol SIT1602BC 12Mhz:SIT1602BC-33-33E-12.000000T -> GP2040-RE:Ocillator; DigiKey Part Number (none) -> 1473-SIT1602BC-33-33E-12.000000-ND
- gave numbers to parts that had none: 1
Connections:
- net +: now also R12.1, U1.47 (USB_DP)
- net +1V1: now also C12.1, C9.1, U1.23 (DVDD), U1.45 (VREG_VOUT), U1.50 (DVDD); no longer C14.1, C4.1
- net +3.3V: now also C14.1, C4.1, R3.2, U1.1 (IOVDD), U1.10 (IOVDD), U1.22 (IOVDD), U1.33 (IOVDD), U1.42 (IOVDD), U1.43 (ADC_AVDD), U1.44 (VREG_VIN), U1.48 (USB_VDD), U1.49 (IOVDD), C13.1, R11.1; no longer C12.1, C9.1, R3.1
- net BlueSolid: now also U1.5 (GPIO3)
- net BlueStripe: now also U1.6 (GPIO4)
- net BrownSolid: now also U1.9 (GPIO7); no longer D3.2
- net BrownStripe: now also U1.8 (GPIO6)
- net CD_gpio: now also U1.36 (GPIO24)
- net CLK_gpio: now also U1.29 (GPIO18)
- net CMD_gpio: now also U1.30 (GPIO19)
- net D0_gpio: now also U1.31 (GPIO20)
- net D1_gpio: now also U1.32 (GPIO21)
- net D2_gpio: now also U1.34 (GPIO22)
- net D3_gpio: now also U1.35 (GPIO23)
- net Data_Command: now also U1.15 (GPIO12)
- net GND: now also U1.19 (TESTEN), U1.21 (XOUT), U1.57 (GND), C13.2, C18.2, J5.3 (Pin_3), R11.2
- net GreenSolid: now also U1.7 (GPIO5)
- net GreenStripe: now also U1.4 (GPIO2)
- net InputVoltage: now also C18.1
- net OCS: now also U1.17 (GPIO14)
- net OrangeSolid: now also D3.2
- net QSPI_SCLK: now also U1.52 (SQPI_SCLK)
- net QSPI_SD0: now also U1.53 (SQPI_SD0)
- net QSPI_SD1: now also U1.55 (SQPI_SD1)
- net QSPI_SD2: now also U1.54 (SQPI_SD2)
- net QSPI_SD3: now also U1.51 (SQPI_SD3)
- net QSPI_SS: now also U1.56 (SQPI_SS_N)
- net RESET: now also U1.16 (GPIO13)
- net RUN: now also U1.26 (RUN)
- net SPI1_RX_MISO: now also U1.11 (GPIO8)
- net SPI1_SCK: now also U1.13 (GPIO10)
- net SPI1_TX_MOSI: now also U1.14 (GPIO11)
- net SWCLK: now also U1.24 (SWCLK)
- net SWDIO: now also U1.25 (SWDIO)
- net VBUS: now also Q1.2 (Collector); no longer Q1.3 (C)
- net XIN: now also U1.20 (XIN)
- net at J8.2 (Pin_2): now also Q1.3 (Emitter); no longer Q1.2 (E)
- net UART_TX: now reaches U1.2 (GPIO0)
- net UART_TX: now also J5.2 (Pin_2)
- net SDA_0: now reaches U1.27 (GPIO16)
- net SDA_0: now also J1.1, R2.1
- net SCL_0: now reaches U1.28 (GPIO17)
- net SCL_0: now also J1.2, R3.1
- net UART_RX: now reaches U1.3 (GPIO1)
- net UART_RX: now also J5.1 (Pin_1)
- net SDA_1: now reaches U1.38 (GPIO26/ADC0)
- net SDA_1: now also J2.1
- net SCL_1: now reaches U1.39 (GPIO27/ADC1)
- net SCL_1: now also J2.2
- net -: now reaches R13.1, U1.46 (USB_DM)
- removed net SCL: J1.2, J2.2, R3.2
- removed net SDA: J1.1, J2.1, R2.1
- no-connect marks 13 -> 10
Other:
- note added: "Additional perhipherals"
- note added: "GP2040-CE connection"
- moved on the sheet: C10, C11, C12, C14, C15, C16, C17, C3, C4, C5, C6, C7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

Commit message: 4 Layer board
Parts:
- C18: DigiKey Part Number (none) -> 1276-CL10A476MQ8QRNCCT-ND
Changed lines of the file:
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@@
+			)
+		)
+		(property "DigiKey Part Number" "1276-CL10A476MQ8QRNCCT-ND"
+			(at 55.88 179.07 0)
+			(effects
+				(font
+					(size 1.27 1.27)
+				)
+				(hide yes)
 			)
 		)

Commit message: What a roller coaster
Parts:
- removed D1, D2: LED_Small, LED_SMD:LED_0603_1608Metric, symbol Device:LED_Small
- removed J2: I2C Controller, GP2040-RE:CONN_SM04B-SRSS-TB_JST, symbol GP2040-RE:qwiic
- removed J4: USB Programming, Connector_PinHeader_2.54mm:PinHeader_1x04_P2.54mm_Vertical, symbol Connector:Conn_01x04_Pin
- removed Q1: NPN 65V 0.1A, GP2040-RE:SOT-323-3_2P2X1P35_ONS, symbol GP2040-RE:FET
- removed R10: 10k, Resistor_SMD:R_0603_1608Metric, symbol Device:R_Small
- removed U5: TPS3702CX50DDCR, GP2040-RE:DDC0006A_N, symbol GP2040-RE:Voltage Supervisor
- added C19: 0.1uF, Capacitor_SMD:C_0603_1608Metric, symbol Device:C_Small
- added C20: 0.1uf, Capacitor_SMD:C_0603_1608Metric, symbol Device:C_Small
- added D5: 20V 1A, GP2040-RE:SDO_SOD-123FL_ONS, symbol GP2040-RE:Schottky
- added H1, H2, H3, H4: MountingHole, MountingHole:MountingHole_2.5mm, symbol Mechanical:MountingHole
- added J2: CONN HEADER R/A 6POS 2.54MM, GP2040-RE:WURTH_61200621721, symbol GP2040-RE:CONN HEADER R/A 6POS 2.54MM
- added J4: GSB1C4621DS2HR, GP2040-RE:AMPHENOL_GSB1C4621DS2HR, symbol GP2040-RE:GSB1C4621DS2HR
- added J9: Conn_01x02, Connector_PinHeader_2.54mm:PinHeader_1x02_P2.54mm_Vertical, symbol Connector_Generic:Conn_01x02
- added R14: 130, Resistor_SMD:R_0603_1608Metric_Pad0.98x0.95mm_HandSolder, symbol Device:R_Small
- added U3: TXB0108PWR, GP2040-RE:TXB0108PWR, symbol GP2040-RE:TXB0108PWR
- R4, R5: value 10k -> 5K1; footprint Resistor_SMD:R_0603_1608Metric -> Resistor_SMD:R_0603_1608Metric_Pad0.98x0.95mm_HandSolder; DigiKey Part Number P10.0KHCT-ND -> (none)
Connections:
- net 5V_EN is gone; now on net GND: R5.1
- net +3.3V: now also J8.2 (Pin_2), C20.2, J2.3, U3.2 (VCCA); no longer R4.1
- net BlueSolid: now also U3.15 (B5); no longer U1.5 (GPIO3)
- net BlueStripe: now also U3.16 (B4); no longer U1.6 (GPIO4)
- net BrownSolid: now also U3.20 (B1); no longer U1.9 (GPIO7)
- net BrownStripe: now also U3.18 (B2); no longer U1.8 (GPIO6)
- net D+: now also J4.A6 (DP1), J4.B6 (DP2)
- net D-: now also J4.A7 (DN1), J4.B7 (DN2)
- net GND: now also R4.2, C19.1, C20.1, J2.4, J4.A1_B12 (GND_A), J4.B1_A12 (GND_B), J4.SH1 (SHIELD), J4.SH2 (SHIELD__1), J4.SH3 (SHIELD__2), J4.SH4 (SHIELD__3), J9.2 (Pin_2), R14.2, U3.11 (GND)
- net GreenSolid: now also U3.17 (B3); no longer U1.7 (GPIO5)
- net GreenStripe: now also U3.14 (B6); no longer U1.4 (GPIO2)
- net InputVoltage: now also C19.2, D5.1, U3.19 (VCCB)
- net RUN: now also J2.5
- net SCL_0: now also J2.2
- net SDA_0: now also J2.1
- net VBUS: now also J4.A4_B9 (VBUS_A), J4.B4_A9 (VBUS_B)
- net at R5.2: now also J4.B5 (CC2)
- new net: R14.1, U3.10 (OE)
- new net: J4.A5 (CC1), R4.1
- new net 3v3BlueSolid: U1.5 (GPIO3), U3.6 (A5)
- new net 3v3BlueStripe: U1.6 (GPIO4), U3.5 (A4)
- new net 3v3BrownSolid: U1.9 (GPIO7), U3.1 (A1)
- new net 3v3BrownStripe: U1.8 (GPIO6), U3.3 (A2)
- new net 3v3GreenSolid: U1.7 (GPIO5), U3.4 (A3)
- new net 3v3GreenStripe: U1.4 (GPIO2), U3.7 (A6)
- new net VCC: D5.2, J2.6, J9.1 (Pin_1)
- no-connect marks 10 -> 16
Other:
- note removed: "Additional perhipherals"
- moved on the sheet: C10, C11, C12, C13, C14, C15, C16, C17, C18, C4, C5, C6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

Commit message: Documentation day
Parts:
- removed U3: TXB0108PWR, GP2040-RE:TXB0108PWR, symbol GP2040-RE:TXB0108PWR
- added U3: TXS0108ERGYR, GP2040-RE:RGY20_3P05X2P05, symbol GP2040-RE:TXS0108ERGYR
- J4: value GSB1C4621DS2HR -> USB4105-GF-A; footprint GP2040-RE:AMPHENOL_GSB1C4621DS2HR -> GP2040-RE:GCT_USB4105-GF-A; symbol GP2040-RE:GSB1C4621DS2HR -> GP2040-RE:USB4105-GF-A; DigiKey Part Number 664-GSB1C4621DS2HRCT-ND -> 2073-USB4105-GF-ACT-ND
Connections:
- net +3.3V: now also U3.2 (VCCA)
- net 3v3BlueSolid: now also U3.7 (A6)
- net 3v3BlueStripe: now also U3.6 (A5)
- net 3v3BrownSolid: now also U3.3 (A2)
- net 3v3BrownStripe: now also U3.4 (A3)
- net 3v3GreenSolid: now also U3.5 (A4)
- net 3v3GreenStripe: now also U3.8 (A7)
- net BlueSolid: now also U3.14 (B6)
- net BlueStripe: now also U3.15 (B5)
- net BrownSolid: now also U3.18 (B2)
- net BrownStripe: now also U3.17 (B3)
- net GND: now also U3.11 (GND), U3.21 (EPAD)
- net GreenSolid: now also U3.16 (B4)
- net GreenStripe: now also U3.13 (B7)
- net InputVoltage: now also U3.19 (VCCB)
- net at R14.1: now also U3.10 (OE)
Other:
- moved on the sheet: C19, C20, J4, R14, R4, R5

Commit message: Updates to PCB and level shifters
Parts:
- removed C15: 100n 6.3V X5R 10%, Capacitor_SMD:C_0603_1608Metric, symbol Device:C_Small
- removed C16, C17, C18: 47u 6.3V X5R 20%, Capacitor_SMD:C_0603_1608Metric, symbol Device:C_Small
- removed C19: 0.1uF, Capacitor_SMD:C_0603_1608Metric, symbol Device:C_Small
- removed C20: 0.1uf, Capacitor_SMD:C_0603_1608Metric, symbol Device:C_Small
- removed D3, D4, D5: 20V 1A, GP2040-RE:SDO_SOD-123FL_ONS, symbol GP2040-RE:Schottky
- removed L1: SRN2512-1R0M, GP2040-RE:IND_SRN2512_BRN, symbol GP2040-RE:SRN2512-1R0M
- removed R14: 130, Resistor_SMD:R_0603_1608Metric_Pad0.98x0.95mm_HandSolder, symbol Device:R_Small
- removed R6, R7, R9: 100K 50mW 1%, Resistor_SMD:R_0603_1608Metric, symbol Device:R_Small
- removed R8: 560K 50mW 1%, Resistor_SMD:R_0603_1608Metric, symbol Device:R_Small
- removed U3: TXS0108ERGYR, GP2040-RE:RGY20_3P05X2P05, symbol GP2040-RE:TXS0108ERGYR
- removed U4: Linear Regulator, GP2040-RE:QFN_4AGQW_RIT, symbol GP2040-RE:Linear Regulator
Connections:
- net 3v3BrownSolid is gone; now on net 3v3BrownStripe: U1.9 (GPIO7)
- net 3v3BlueSolid: now also U1.6 (GPIO4); no longer U1.5 (GPIO3)
- net 3v3BlueStripe: now also U1.7 (GPIO5); no longer U1.6 (GPIO4)
- net 3v3BrownStripe: no longer U1.8 (GPIO6)
- net 3v3GreenSolid: now also U1.8 (GPIO6); no longer U1.7 (GPIO5)
- net 3v3GreenStripe: now also U1.5 (GPIO3); no longer U1.4 (GPIO2)
- new net 3v3OrangeSolid: U1.4 (GPIO2)
- no-connect marks 16 -> 11
Other:
- added sheet NES_SNES (NES_SNES.kicad_sch)
- added sheet PowerManagement (Power.kicad_sch)

Commit message: Some code cleanup
Parts:
- added C15: 100n 6.3V X5R 10%, Capacitor_SMD:C_0402_1005Metric_Pad0.74x0.62mm_HandSolder, symbol Device:C_Small
- added C16, C17, C18: 47u 6.3V X5R 20%, Capacitor_SMD:C_0603_1608Metric_Pad1.08x0.95mm_HandSolder, symbol Device:C_Small
- added D1, D2, D3: 20V 1A, GP2040-RE:SDO_SOD-123FL_ONS, symbol GP2040-RE:Schottky
- added L1: 1uH, GP2040-RE:IND_SRN2512_BRN, symbol GP2040-RE:SRN2512-1R0M
- added Q1, Q2, Q3, Q4, Q5, Q6: BSS138, Package_TO_SOT_SMD:SOT-23, symbol Transistor_FET:BSS138
- added R10, R14, R8: 100K 50mW 1%, Resistor_SMD:R_0402_1005Metric_Pad0.72x0.64mm_HandSolder, symbol Device:R_Small
- added R15, R16, R17, R18, R19, R20, R21, R22, R23, R24, R6, R7: 10K, Resistor_SMD:R_0402_1005Metric_Pad0.72x0.64mm_HandSolder, symbol Device:R_Small
- added R9: 560K 50mW 1%, Resistor_SMD:R_0402_1005Metric_Pad0.72x0.64mm_HandSolder, symbol Device:R_Small
- added U3: Linear Regulator, GP2040-RE:QFN_4AGQW_RIT, symbol GP2040-RE:Linear Regulator
- C1, C10, C11, C12, C13, C14, C2, C3, C4, C5, C6, C7, C8, C9: footprint Capacitor_SMD:C_0603_1608Metric -> Capacitor_SMD:C_0402_1005Metric_Pad0.74x0.62mm_HandSolder
- R1, R12, R13, R2, R3: footprint Resistor_SMD:R_0603_1608Metric -> Resistor_SMD:R_0402_1005Metric_Pad0.72x0.64mm_HandSolder
- R4, R5: footprint Resistor_SMD:R_0603_1608Metric_Pad0.98x0.95mm_HandSolder -> Resistor_SMD:R_0402_1005Metric_Pad0.72x0.64mm_HandSolder
Connections:
- net +3.3V: now also C7.2, C16.1, C18.1, Q1.1 (G), Q2.1 (G), Q3.1 (G), Q4.1 (G), Q5.1 (G), Q6.1 (G), R15.1, R17.1, R19.1, R21.1, R23.1, R6.1, R9.1, U3.4 (VOUT), U3.5 (VOUT); no longer C7.1
- net 3v3BlueSolid: now also Q3.2 (S), R17.2
- net 3v3BlueStripe: now also Q4.2 (S), R19.2
- net 3v3BrownStripe: now also Q6.2 (S), R23.2
- net 3v3GreenSolid: now also Q5.2 (S), R21.2
- net 3v3GreenStripe: now also Q2.2 (S), R15.2
- net 3v3OrangeSolid: now also Q1.2 (S), R6.2
- net BlueSolid: now also Q3.3 (D), R18.2
- net BlueStripe: now also Q4.3 (D), R20.2
- net BrownSolid: now also D2.2, R16.1, R18.1, R20.1, R22.1, R24.1, R7.1
- net BrownStripe: now also Q6.3 (D), R24.2
- net GND: now also C7.1, C15.1, C16.2, C17.2, C18.2, R14.2, R8.1, U3.15 (PGND), U3.2 (GND); no longer C7.2
- net GreenSolid: now also Q5.3 (D), R22.2
- net GreenStripe: now also Q2.3 (D), R16.2
- net OrangeSolid: now also Q1.3 (D), R7.2
- net VBUS: now also D3.2
- net VCC: now also D1.2
- new net: C17.1, D1.1, D2.1, D3.1, R10.2, U3.10 (VIN), U3.11 (VIN)
- new net: C15.2, U3.1 (VINA)
- new net: R10.1, U3.12 (EN)
- new net: R8.2, U3.13 (PS/SYNC)
- new net: R14.1, R9.2, U3.3 (FB)
- new net: L1.1, U3.6 (LX2), U3.7 (LX2)
- new net: L1.2, U3.8 (LX1), U3.9 (LX1)
- no-connect marks 11 -> 12
Other:
- removed sheet NES_SNES
- removed sheet PowerManagement
- note added: "3v3 Regulation for RP2040"
- moved on the sheet: C10, C11, C12, C13, C14, C4, C5, C6, C7, C8, C9, J4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
