File: GP2040-RE/GP2040-RE.kicad_pcb (KiCad board)
At the start: 4 copper layers, 63.2 x 36.1 mm, 52 parts, among them J1 I2C Target, J2 I2C Controller, J3 SM03B-SRSS-TB_LF__SN_, J4 USB Programming, J5 Conn_01x03, J6 microSD, J7 RJ-45, J8 Conn_01x10, Q1 NPN 65V 0.1A, U1 RP2040, U2 16M, U4 Linear Regulator, U5 TPS3702CX50DDCR

Commit message: 4 Layer board
Changed lines of the file:
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@@
 			(outputformat 1)
 			(mirror no)
-			(drillshape 1)
+			(drillshape 0)
 			(scaleselection 1)
-			(outputdirectory "")
+			(outputdirectory "Gerbers/")
 		)
 	)
@@
 		(tags "capacitor")
 		(property "Reference" "C1"
-			(at 0 -1.43 270)
+			(at 0 -1.43 -90)
 			(layer "F.SilkS")
 			(effects
@@
 		)
 		(property "Value" "2.2u 6.3V X5R 20%"
-			(at 0 1.43 270)
+			(at 0 1.43 -90)
 			(layer "F.Fab")
 			(effects
@@
 		)
 		(fp_text user "${REFERENCE}"
-			(at 0 0 270)
+			(at 0 0 -90)
 			(layer "F.Fab")
 			(effects
@@
 		(tags "capacitor")
 		(property "Reference" "C17"
-			(at 0 -1.43 270)
+			(at 0 -1.43 -90)
 			(layer "F.SilkS")
 			(effects
@@
 		)
 		(property "Value" "47u 6.3V X5R 20%"
-			(at 0 1.43 270)
+			(at 0 1.43 -90)
 			(layer "F.Fab")
 			(effects
@@
 		)
 		(fp_text user "${REFERENCE}"
-			(at 0 0 270)
+			(at 0 0 -90)
 			(layer "F.Fab")
 			(effects
@@
 		(tags "Through hole pin header THT 1x10 2.54mm single row")
 		(property "Reference" "J8"
-			(at 0 -2.33 270)
+			(at 0 -2.33 -90)
 			(layer "F.SilkS")
 			(effects
@@
 		)
 		(property "Value" "Conn_01x10"
-			(at 0 25.19 270)
+			(at 0 25.19 -90)
 			(layer "F.Fab")
 			(effects
@@
 		)
 		(fp_text user "${REFERENCE}"
-			(at 0 11.43 360)
+			(at 0 11.43 0)
 			(layer "F.Fab")
 			(effects
@@
 		(tags "capacitor")
 		(property "Reference" "C12"
-			(at 0 -2.446 270)
+			(at 0 -2.446 -90)
 			(layer "F.SilkS")
 			(effects
@@
 		)
 		(property "Value" "2.2u 6.3V X5R 20%"
-			(at 0 1.43 270)
+			(at 0 1.43 -90)
 			(layer "F.Fab")
 			(effects
@@
 		)
 		(fp_text user "${REFERENCE}"
-			(at 0 0 270)
+			(at 0 0 -90)
 			(layer "F.Fab")
 			(effects
@@
 		(tags "resistor")
 		(property "Reference" "R7"
-			(at 0 -1.43 270)
+			(at 0 -1.43 -90)
 			(layer "F.SilkS")
 			(effects
@@
 		)
 		(property "Value" "100K 50mW 1%"
-			(at 0 1.43 270)
+			(at 0 1.43 -90)
 			(layer "F.Fab")
 			(effects
@@
 		)
 		(fp_text user "${REFERENCE}"
-			(at 0 0 270)
+			(at 0 0 -90)
 			(layer "F.Fab")
 			(effects
@@
 		(tags "capacitor")
 		(property "Reference" "C2"
-			(at 0 -1.43 270)
+			(at 0 -1.43 -90)
 			(layer "F.SilkS")
 			(effects
@@
 		)
 		(property "Value" "100n 6.3V X5R 10%"
-			(at 0 1.43 270)
+			(at 0 1.43 -90)
 			(layer "F.Fab")
 			(effects
@@
 		)
 		(fp_text user "${REFERENCE}"
-			(at 0 0 270)
+			(at 0 0 -90)
 			(layer "F.Fab")
 			(effects
@@
 		(at 91.186 79.248 90)
 		(property "Reference" "S2"
-			(at 0.55069 -2.13777 270)
+			(at 0.55069 -2.13777 -90)
 			(layer "F.SilkS")
 			(effects
@@
 		)
 		(property "Value" "Buttons"
-			(at 7.54882 2.369355 270)
+			(at 7.54882 2.369355 -90)
 			(layer "F.Fab")
 			(effects
@@
 		(tags "capacitor")
 		(property "Reference" "C10"
-			(at 0 -1.43 270)
+			(at 0 -1.43 -90)
 			(layer "F.SilkS")
 			(effects
@@
 		)
 		(property "Value" "100n 6.3V X5R 10%"
-			(at 0 1.43 270)
+			(at 0 1.43 -90)
 			(layer "F.Fab")
 			(effects
@@
 		)
 		(fp_text user "${REFERENCE}"
-			(at 0 0 270)
+			(at 0 0 -90)
 			(layer "F.Fab")
 			(effects
@@
 		(tags "capacitor")
 		(property "Reference" "C11"
-			(at 0 -1.43 270)
+			(at 0 -1.43 -90)
 			(layer "F.SilkS")
 			(effects
@@
 		)
 		(property "Value" "100n 6.3V X5R 10%"
-			(at 0 1.43 270)
+			(at 0 1.43 -90)
 			(layer "F.Fab")
 			(effects
@@
 		)
 		(fp_text user "${REFERENCE}"
-			(at 0 0 270)
+			(at 0 0 -90)
 			(layer "F.Fab")
 			(effects
@@
 		(tags "capacitor")
 		(property "Reference" "C14"
-			(at 1.257 1.524 270)
+			(at 1.257 1.524 -90)
 			(layer "F.SilkS")
 			(effects
@@
 		)
 		(property "Value" "2.2u 6.3V X5R 20%"
-			(at 0 1.43 270)
+			(at 0 1.43 -90)
 			(layer "F.Fab")
 			(effects
@@
 		)
 		(fp_text user "${REFERENCE}"
-			(at 0 0 270)
+			(at 0 0 -90)
 			(layer "F.Fab")
 			(effects
@@
 		(tags "resistor")
 		(property "Reference" "R12"
-			(at 0 -1.43 270)
+			(at 0 -1.43 -90)
 			(layer "F.SilkS")
 			(effects
@@
 		)
 		(property "Value" "27 50mW 1% M0603"
-			(at 0 1.43 270)
+			(at 0 1.43 -90)
 			(layer "F.Fab")
 			(effects
@@
 		)
 		(fp_text user "${REFERENCE}"
-			(at 0 0 270)
+			(at 0 0 -90)
 			(layer "F.Fab")
 			(effects
@@
 		(tags "capacitor")
 		(property "Reference" "C16"
-			(at 0 -1.43 270)
+			(at 0 -1.43 -90)
 			(layer "F.SilkS")
 			(effects
@@
 		)
 		(property "Value" "47u 6.3V X5R 20%"
-			(at 0 1.43 270)
+			(at 0 1.43 -90)
 			(layer "F.Fab")
 			(effects
@@
 		)
 		(fp_text user "${REFERENCE}"
-			(at 0 0 270)
+			(at 0 0 -90)
 			(layer "F.Fab")
 			(effects
@@
 		(at 93.472 79.248 90)
 		(property "Reference" "S1"
-			(at 0.55069 -2.13777 270)
+			(at 0.55069 -2.13777 -90)
 			(layer "F.SilkS")
 			(effects
@@
 		)
 		(property "Value" "Buttons"
-			(at 7.54882 2.369355 270)
+			(at 7.54882 2.369355 -90)
 			(layer "F.Fab")
 			(effects
@@
 		(tags "resistor")
 		(property "Reference" "R13"
-			(at 0 -1.43 270)
+			(at 0 -1.43 -90)
 			(layer "F.SilkS")
 			(effects
@@
 		)
 		(property "Value" "27 50mW 1% M0603"
-			(at 0 1.43 270)
+			(at 0 1.43 -90)
 			(layer "F.Fab")
 			(effects
@@
 		)
 		(fp_text user "${REFERENCE}"
-			(at 0 0 270)
+			(at 0 0 -90)
 			(layer "F.Fab")
 			(effects
@@
 		(tags "capacitor")
 		(property "Reference" "C18"
-			(at 0 -1.43 270)
+			(at 0 -1.43 -90)
 			(layer "F.SilkS")
 			(effects
@@
 		)
 		(property "Value" "47u 6.3V X5R 20%"
-			(at 0 1.43 270)
+			(at 0 1.43 -90)
 			(layer "F.Fab")
 			(effects
@@
 		)
 		(fp_text user "${REFERENCE}"
-			(at 0 0 270)
+			(at 0 0 -90)
 			(layer "F.Fab")
 			(effects
@@
 		(tags "resistor")
 		(property "Reference" "R2"
-			(at 0 -1.43 360)
+			(at 0 -1.43 0)
 			(layer "F.SilkS")
 			(effects
@@
 		)
 		(property "Value" "4.7k"
-			(at 0 1.43 360)
+			(at 0 1.43 0)
 			(layer "F.Fab")
 			(effects
@@
 		)
 		(fp_text user "${REFERENCE}"
-			(at 0 0 360)
+			(at 0 0 0)
 			(layer "F.Fab")
 			(effects
@@
 		(pts
 			(xy 65.532 74.422) (xy 66.294 74.422) (xy 66.548 74.168) (xy 66.548 73.914) (xy 68.834 73.914) (xy 69.342 73.914)
-			(xy 69.342 74.93) (xy 69.342 74.93) (xy 65.532 74.93)
+			(xy 69.342 74.93) (xy 65.532 74.93)
 		)
 		(stroke

Commit message: What a roller coaster
Parts:
- removed D1, D2: LED_Small, LED_SMD:LED_0603_1608Metric
- removed Q1: NPN 65V 0.1A, GP2040-RE:SOT-323-3_2P2X1P35_ONS
- removed R10: 10k, Resistor_SMD:R_0603_1608Metric
- removed U5: TPS3702CX50DDCR, GP2040-RE:DDC0006A_N
- added C19: 0.1uF, Capacitor_SMD:C_0603_1608Metric, F.Cu at (114.2, 90.2)
- added C20: 0.1uf, Capacitor_SMD:C_0603_1608Metric, F.Cu at (126.5, 90.8)
- added D5: 20V 1A, GP2040-RE:SDO_SOD-123FL_ONS, F.Cu at (107.8, 101.8)
- added H1: MountingHole, MountingHole:MountingHole_2.5mm, F.Cu at (152.7, 76.2)
- added H2: MountingHole, MountingHole:MountingHole_2.5mm, F.Cu at (152.4, 101.3)
- added H3: MountingHole, MountingHole:MountingHole_2.5mm, F.Cu at (101.6, 101.9)
- added H4: MountingHole, MountingHole:MountingHole_2.5mm, F.Cu at (101.6, 76.2)
- added J9: Conn_01x02, Connector_PinHeader_2.54mm:PinHeader_1x02_P2.54mm_Vertical, F.Cu at (112.1, 101.8)
- added R14: 130, Resistor_SMD:R_0603_1608Metric_Pad0.98x0.95mm_HandSolder, F.Cu at (126.7, 82.4)
- added U3: TXB0108PWR, GP2040-RE:TXB0108PWR, F.Cu at (120.0, 87.2)
- J2: value I2C Controller -> CONN HEADER R/A 6POS 2.54MM; footprint GP2040-RE:CONN_SM04B-SRSS-TB_JST -> GP2040-RE:WURTH_61200621721
- J4: value USB Programming -> GSB1C4621DS2HR; footprint Connector_PinHeader_2.54mm:PinHeader_1x04_P2.54mm_Vertical -> GP2040-RE:AMPHENOL_GSB1C4621DS2HR
- R4, R5: value 10k -> 5K1; footprint Resistor_SMD:R_0603_1608Metric -> Resistor_SMD:R_0603_1608Metric_Pad0.98x0.95mm_HandSolder
- moved J2 103.6 mm to (165.4, 88.1), turned to 90 degrees
- moved J8 96.7 mm to (157.9, 99.3), turned to 180 degrees
- moved S2 73.6 mm to (164.6, 74.0), turned to 180 degrees
- moved S1 71.5 mm to (164.6, 71.9), turned to 180 degrees
- moved J4 62.3 mm to (142.2, 70.4), turned to 180 degrees
- moved R12 60.9 mm to (138.0, 79.1), turned to 0 degrees
- moved R13 60.0 mm to (138.0, 80.7), turned to 0 degrees
- moved C1 59.8 mm to (130.0, 77.5)
- moved C2 59.7 mm to (131.5, 77.5)
- moved C14 59.4 mm to (140.2, 81.4)
- moved R11 59.3 mm to (143.5, 84.7), turned to -90 degrees
- moved C12 59.0 mm to (138.0, 82.2), turned to 0 degrees
- moved C10 57.3 mm to (134.5, 79.6)
- moved C11 57.3 mm to (133.0, 79.6)
- moved R1 56.9 mm to (126.2, 74.8), turned to 180 degrees
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Connections:
- J2 pad 1: /SDA_1 -> /SDA_0
- J2 pad 2: /SCL_1 -> /SCL_0
- J2 pad 5: (no net) -> /RUN
- J2 pad 6: (no net) -> VCC
- J8 pad 2: Net-(J8-Pin_2) -> +3.3V
- R4 pad 1: +3.3V -> Net-(J4-CC1)
- R4 pad 2: Net-(D1-A) -> GND
- R5 pad 1: /5V_EN -> GND
- R5 pad 2: Net-(D2-A) -> Net-(J4-CC2)
- U1 pad 4: /GreenStripe -> /3v3GreenStripe
- U1 pad 5: /BlueSolid -> /3v3BlueSolid
- U1 pad 6: /BlueStripe -> /3v3BlueStripe
- U1 pad 7: /GreenSolid -> /3v3GreenSolid
- U1 pad 8: /BrownStripe -> /3v3BrownStripe
- U1 pad 9: /BrownSolid -> /3v3BrownSolid
Routing:
- net VCC: track 0.00 -> 62.7 mm
- net /SCL_1: track 52.6 -> 1.11 mm, vias 2 -> 1
- net /SDA_1: track 50.5 -> 1.06 mm, vias 2 -> 1
- net /RUN: track 12.4 -> 58.0 mm, vias 0 -> 1
- net /5V_EN: track 42.7 -> 0.00 mm, vias 2 -> 0
- net /InputVoltage: track 10.1 -> 36.1 mm
- net /SPI1_SCK: track 56.7 -> 31.6 mm
- net /OCS: track 52.5 -> 27.8 mm
- net /RESET: track 52.7 -> 29.5 mm
- net /Data_Command: track 53.9 -> 31.2 mm
- net /SPI1_TX_MOSI: track 57.1 -> 37.0 mm
- net /SPI1_RX_MISO: track 58.1 -> 38.4 mm
- net /SDA_0: track 61.6 -> 78.7 mm
- net /SCL_0: track 65.2 -> 81.0 mm
- net /UART_RX: track 18.3 -> 29.7 mm, vias 1 -> 2
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Other:
- board size 63.2 x 36.1 mm -> 88.4 x 36.1 mm

Commit message: Documentation day
Parts:
- J4: value GSB1C4621DS2HR -> USB4105-GF-A; footprint GP2040-RE:AMPHENOL_GSB1C4621DS2HR -> GP2040-RE:GCT_USB4105-GF-A
- U3: value TXB0108PWR -> TXS0108ERGYR; footprint GP2040-RE:TXB0108PWR -> GP2040-RE:RGY20_3P05X2P05
- moved R14 23.5 mm to (103.2, 81.2), turned to 180 degrees
- moved U3 16.9 mm to (103.2, 85.3)
- moved J2 11.8 mm to (153.5, 88.1)
- moved S1 11.7 mm to (153.7, 76.0)
- moved S2 11.7 mm to (153.6, 78.2)
- moved J8 11.0 mm to (146.9, 99.3)
- moved H1 10.3 mm to (142.4, 76.1)
- moved H2 10.0 mm to (142.4, 101.8)
- moved J4 7.79 mm to (134.4, 70.3)
- moved U1 7.44 mm to (125.9, 87.1)
- moved XTAL1 7.44 mm to (121.2, 93.9)
- moved C1 7.44 mm to (122.6, 77.5)
- moved C10 7.44 mm to (127.1, 79.6)
- moved C11 7.44 mm to (125.5, 79.6)
- moved C12 7.44 mm to (130.5, 82.2)
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Connections:
- U3 pad 1: /3v3BrownSolid -> unconnected-(U3-A1-Pad1)
- U3 pad 13: unconnected-(U3-B7-Pad13) -> /GreenStripe
- U3 pad 14: /GreenStripe -> /BlueSolid
- U3 pad 15: /BlueSolid -> /BlueStripe
- U3 pad 16: /BlueStripe -> /GreenSolid
- U3 pad 17: /GreenSolid -> /BrownStripe
- U3 pad 18: /BrownStripe -> /BrownSolid
- U3 pad 20: /BrownSolid -> unconnected-(U3-B1-Pad20)
- U3 pad 3: /3v3BrownStripe -> /3v3BrownSolid
- U3 pad 4: /3v3GreenSolid -> /3v3BrownStripe
- U3 pad 5: /3v3BlueStripe -> /3v3GreenSolid
- U3 pad 6: /3v3BlueSolid -> /3v3BlueStripe
- U3 pad 7: /3v3GreenStripe -> /3v3BlueSolid
- U3 pad 8: unconnected-(U3-A7-Pad8) -> /3v3GreenStripe
Routing:
- net +3.3V: track 61.5 -> 86.9 mm, vias 13 -> 11
- net /D1_gpio: track 81.3 -> 59.6 mm
- net /D0_gpio: track 80.2 -> 58.5 mm
- net /SDA_0: track 78.7 -> 60.2 mm
- net /SCL_0: track 81.0 -> 65.0 mm, vias 2 -> 3
- net /CLK_gpio: track 75.2 -> 60.6 mm
- net /CMD_gpio: track 74.2 -> 59.7 mm
- net /GreenStripe: track 25.1 -> 11.9 mm, vias 1 -> 0
- net /CD_gpio: track 61.1 -> 48.2 mm
- net /D3_gpio: track 65.1 -> 53.1 mm
- net /BlueStripe: track 25.6 -> 14.1 mm, vias 1 -> 0
- net /GreenSolid: track 23.3 -> 12.3 mm, vias 1 -> 0
- net /3v3GreenStripe: track 7.26 -> 18.2 mm
- net /3v3BlueSolid: track 7.36 -> 18.2 mm
- net /3v3BlueStripe: track 7.47 -> 18.1 mm
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Other:
- board size 88.4 x 36.1 mm -> 77.7 x 36.1 mm
- board text added: "3v3"
- board text added: "BOOT"
- board text added: "Blue Solid"
- board text added: "Blue Stripe"
- board text added: "Brown Solid"
- board text added: "Brown Stripe"
- board text added: "CLK"
- board text added: "DC"
- board text added: "Designed by Fortinbra"
- board text added: "G"
- board text added: "GND"
- board text added: "Green Solid"
- board text added: "Green Stripe"
- board text added: "Ground"
- board text added: "MISO"
- board text added: "MOSI"
- board text added: "NC"
- board text added: "OCS"
- board text added: "Oragne Solid"
- board text added: "Orange Solid"
- board text added: "Orange Stripe"
- board text added: "Orange Stripe = Ground Orange Solid = SNES 5V Green Strip = SNES Data 2 (Unused) Blue Solid = SNES Data 0 Blue Stripe = SNES Data 1 (Unused) Green Solid = SNES Latch Brown Stripe = Unused Brown Solid = SNES Clock"
- board text added: "RE"
- board text added: "RESET"
- board text added: "RUN"
- board text added: "RX"
- board text added: "SCL 0"
- board text added: "SDA 0"
- board text added: "SWCLK"
- board text added: "SWDIO"
- board text added: "T568B"
- board text added: "TX"
- board text added: "UART"
- board text added: "VCC"
- board text added: "qwiic SDA/SCL 0"

Commit message: Updates to PCB and level shifters
Routing:
- net +1V1: track 22.5 -> 21.3 mm
- net /SWCLK: track 10.1 -> 9.56 mm
