File: GP2040-RE/GP2040-RE.kicad_pcb (KiCad board)
At the start: 4 copper layers, 77.7 x 36.1 mm, 57 parts, among them J1 I2C Target, J2 CONN HEADER R/A 6POS 2.54MM, J3 SM03B-SRSS-TB_LF__SN_, J4 USB4105-GF-A, J5 Conn_01x03, J6 microSD, J7 RJ-45, J8 Conn_01x10, J9 Conn_01x02, U1 RP2040, U2 16M, U3 TXS0108ERGYR, U4 Linear Regulator

Commit message: Some code cleanup
Parts:
- removed C19: 0.1uF, Capacitor_SMD:C_0603_1608Metric
- removed C20: 0.1uf, Capacitor_SMD:C_0603_1608Metric
- removed D4, D5: 20V 1A, GP2040-RE:SDO_SOD-123FL_ONS
- removed U4: Linear Regulator, GP2040-RE:QFN_4AGQW_RIT
- added D1: 20V 1A, GP2040-RE:SDO_SOD-123FL_ONS, F.Cu at (110.3, 101.6)
- added D2: 20V 1A, GP2040-RE:SDO_SOD-123FL_ONS, F.Cu at (110.3, 99.2)
- added Q1: BSS138, Package_TO_SOT_SMD:SOT-23, F.Cu at (103.3, 79.8)
- added Q2: BSS138, Package_TO_SOT_SMD:SOT-23, F.Cu at (103.3, 83.2)
- added Q3: BSS138, Package_TO_SOT_SMD:SOT-23, F.Cu at (103.3, 86.6)
- added Q4: BSS138, Package_TO_SOT_SMD:SOT-23, F.Cu at (103.3, 90.1)
- added Q5: BSS138, Package_TO_SOT_SMD:SOT-23, F.Cu at (103.3, 93.5)
- added Q6: BSS138, Package_TO_SOT_SMD:SOT-23, F.Cu at (103.3, 96.9)
- added R10: 100K 50mW 1%, Resistor_SMD:R_0402_1005Metric_Pad0.72x0.64mm_HandSolder, F.Cu at (110.8, 95.7)
- added R15: 10K, Resistor_SMD:R_0402_1005Metric_Pad0.72x0.64mm_HandSolder, F.Cu at (105.7, 83.2)
- added R16: 10K, Resistor_SMD:R_0402_1005Metric_Pad0.72x0.64mm_HandSolder, F.Cu at (100.9, 82.7)
- added R17: 10K, Resistor_SMD:R_0402_1005Metric_Pad0.72x0.64mm_HandSolder, F.Cu at (105.7, 86.6)
- added R18: 10K, Resistor_SMD:R_0402_1005Metric_Pad0.72x0.64mm_HandSolder, F.Cu at (100.9, 87.2)
- added R19: 10K, Resistor_SMD:R_0402_1005Metric_Pad0.72x0.64mm_HandSolder, F.Cu at (105.7, 90.0)
- added R20: 10K, Resistor_SMD:R_0402_1005Metric_Pad0.72x0.64mm_HandSolder, F.Cu at (100.9, 89.5)
- added R21: 10K, Resistor_SMD:R_0402_1005Metric_Pad0.72x0.64mm_HandSolder, F.Cu at (105.7, 93.4)
- added R22: 10K, Resistor_SMD:R_0402_1005Metric_Pad0.72x0.64mm_HandSolder, F.Cu at (100.9, 94.1)
- added R23: 10K, Resistor_SMD:R_0402_1005Metric_Pad0.72x0.64mm_HandSolder, F.Cu at (105.7, 96.8)
- added R24: 10K, Resistor_SMD:R_0402_1005Metric_Pad0.72x0.64mm_HandSolder, F.Cu at (100.9, 96.3)
- C1, C10, C11, C12, C13, C14, C15, C2, C3, C4, C5, C6, C7, C8, C9: footprint Capacitor_SMD:C_0603_1608Metric -> Capacitor_SMD:C_0402_1005Metric_Pad0.74x0.62mm_HandSolder
- C16, C17, C18: footprint Capacitor_SMD:C_0603_1608Metric -> Capacitor_SMD:C_0603_1608Metric_Pad1.08x0.95mm_HandSolder
- L1: value SRN2512-1R0M -> 1uH
- R1, R12, R13, R2, R3: footprint Resistor_SMD:R_0603_1608Metric -> Resistor_SMD:R_0402_1005Metric_Pad0.72x0.64mm_HandSolder
- R14: value 130 -> 100K 50mW 1%; footprint Resistor_SMD:R_0603_1608Metric_Pad0.98x0.95mm_HandSolder -> Resistor_SMD:R_0402_1005Metric_Pad0.72x0.64mm_HandSolder
- R4, R5: footprint Resistor_SMD:R_0603_1608Metric_Pad0.98x0.95mm_HandSolder -> Resistor_SMD:R_0402_1005Metric_Pad0.72x0.64mm_HandSolder
- R6, R7: value 100K 50mW 1% -> 10K; footprint Resistor_SMD:R_0603_1608Metric -> Resistor_SMD:R_0402_1005Metric_Pad0.72x0.64mm_HandSolder
- R8: value 560K 50mW 1% -> 100K 50mW 1%; footprint Resistor_SMD:R_0603_1608Metric -> Resistor_SMD:R_0402_1005Metric_Pad0.72x0.64mm_HandSolder
- R9: value 100K 50mW 1% -> 560K 50mW 1%; footprint Resistor_SMD:R_0603_1608Metric -> Resistor_SMD:R_0402_1005Metric_Pad0.72x0.64mm_HandSolder
- U3: value TXS0108ERGYR -> Linear Regulator; footprint GP2040-RE:RGY20_3P05X2P05 -> GP2040-RE:QFN_4AGQW_RIT
- moved S1 28.6 mm to (125.1, 73.9)
- moved S2 28.6 mm to (125.1, 76.1)
- moved R14 19.7 mm to (116.3, 95.8), turned to 0 degrees
- moved R6 19.2 mm to (105.7, 79.8), turned to 90 degrees
- moved R7 16.3 mm to (100.9, 80.4)
- moved D3 16.1 mm to (116.1, 98.6), turned to 0 degrees
- moved U3 14.0 mm to (113.4, 94.9)
- moved H1 12.4 mm to (154.7, 74.7)
- moved H2 12.3 mm to (154.7, 101.6)
- moved C18 11.2 mm to (116.9, 93.6), turned to 0 degrees
- moved R5 6.51 mm to (135.9, 81.1), turned to 90 degrees
- moved R12 6.50 mm to (124.9, 82.3), turned to 90 degrees
- moved C14 5.07 mm to (127.8, 82.3)
- moved J4 5.06 mm to (137.4, 74.4)
- moved R8 5.01 mm to (109.3, 95.7), turned to 90 degrees
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Connections:
- C15 pad 1: Net-(U4-VINA) -> GND
- C15 pad 2: GND -> Net-(U3-VINA)
- C17 pad 1: +3.3V -> Net-(C17-Pad1)
- C18 pad 1: /InputVoltage -> +3.3V
- C7 pad 1: +3.3V -> GND
- C7 pad 2: GND -> +3.3V
- D3 pad 1: /InputVoltage -> Net-(C17-Pad1)
- D3 pad 2: /OrangeSolid -> VBUS
- R14 pad 1: Net-(U3-OE) -> Net-(U3-FB)
- R6 pad 1: Net-(U4-PS/SYNC) -> +3.3V
- R6 pad 2: GND -> /3v3OrangeSolid
- R7 pad 1: Net-(U4-EN) -> /BrownSolid
- R7 pad 2: /InputVoltage -> /OrangeSolid
- R8 pad 1: +3.3V -> GND
- R8 pad 2: Net-(U4-FB) -> Net-(U3-PS/SYNC)
- R9 pad 1: Net-(U4-FB) -> +3.3V
- R9 pad 2: GND -> Net-(U3-FB)
- U1 pad 4: /3v3GreenStripe -> /3v3OrangeSolid
- U1 pad 5: /3v3BlueSolid -> /3v3GreenStripe
- U1 pad 6: /3v3BlueStripe -> /3v3BlueSolid
- U1 pad 7: /3v3GreenSolid -> /3v3BlueStripe
- U1 pad 8: /3v3BrownStripe -> /3v3GreenSolid
- U1 pad 9: /3v3BrownSolid -> /3v3BrownStripe
- U3 pad 1: unconnected-(U3-A1-Pad1) -> Net-(U3-VINA)
- U3 pad 10: Net-(U3-OE) -> Net-(C17-Pad1)
- U3 pad 11: GND -> Net-(C17-Pad1)
- U3 pad 12: unconnected-(U3-B8-Pad12) -> Net-(U3-EN)
- U3 pad 13: /GreenStripe -> Net-(U3-PS/SYNC)
- U3 pad 14: /BlueSolid -> unconnected-(U3-PGOOD-Pad14)
- U3 pad 15: /BlueStripe -> GND
- U3 pad 2: +3.3V -> GND
- U3 pad 3: /3v3BrownSolid -> Net-(U3-FB)
- U3 pad 4: /3v3BrownStripe -> +3.3V
- U3 pad 5: /3v3GreenSolid -> +3.3V
- U3 pad 6: /3v3BlueStripe -> Net-(L1-Pad1)
- U3 pad 7: /3v3BlueSolid -> Net-(L1-Pad1)
- U3 pad 8: /3v3GreenStripe -> Net-(L1-Pad2)
- U3 pad 9: unconnected-(U3-A8-Pad9) -> Net-(L1-Pad2)
Routing:
- net +3.3V: track 86.9 -> 0.00 mm, vias 11 -> 0
- net GND: track 77.0 -> 0.00 mm, vias 34 -> 0
- net /SCL_0: track 65.0 -> 0.00 mm, vias 3 -> 0
- net /CLK_gpio: track 60.6 -> 0.00 mm, vias 2 -> 0
- net /SDA_0: track 60.2 -> 0.00 mm, vias 2 -> 0
- net /CMD_gpio: track 59.7 -> 0.00 mm, vias 2 -> 0
- net /D1_gpio: track 59.6 -> 0.00 mm, vias 2 -> 0
- net /D0_gpio: track 58.5 -> 0.00 mm, vias 2 -> 0
- net VBUS: track 55.1 -> 0.00 mm, vias 2 -> 0
- net /D2_gpio: track 54.0 -> 0.00 mm, vias 2 -> 0
- net VCC: track 53.9 -> 0.00 mm
- net /D3_gpio: track 53.1 -> 0.00 mm, vias 2 -> 0
- net /RUN: track 52.0 -> 0.00 mm
- net /CD_gpio: track 48.2 -> 0.00 mm, vias 2 -> 0
- net /InputVoltage: track 44.5 -> 0.00 mm, vias 2 -> 0
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Other:
- board size 77.7 x 36.1 mm -> 77.7 x 33 mm

Commit message: sync
Parts:
- moved C13 0.97 mm to (128.7, 82.3)
Routing:
- net +3.3V: track 0.00 -> 24.8 mm, vias 0 -> 8
- net GND: track 0.00 -> 12.2 mm, vias 0 -> 6
- net /QSPI_SD3: track 0.00 -> 5.48 mm
- net +1V1: track 0.00 -> 4.40 mm
- net /QSPI_SS: track 0.00 -> 2.56 mm
- net /-: track 0.00 -> 1.90 mm
- net /+: track 0.00 -> 1.89 mm
